Commit message: URDF Update

File: turtlebot3_manipulation/turtlebot3_manipulation_description/xacro/open_manipulator_x.urdf.xacro (robot description, xacro)
@@ -6,5 +6,5 @@
 -->
 <robot xmlns:xacro="http://www.ros.org/wiki/xacro">
-  <xacro:macro name="open_manipulator_x" params="prefix">
+  <xacro:macro name="open_manipulator_x" params="prefix visual_material:=grey show_tool_marker:=true">
     <xacro:property
       name="meshes_file_direction"
@@ -16,5 +16,5 @@
           <mesh filename="${meshes_file_direction}/link1.stl" scale="0.001 0.001 0.001"/>
         </geometry>
-        <material name="grey"/>
+        <material name="${visual_material}"/>
       </visual>
       <collision>
@@ -46,5 +46,5 @@
           <mesh filename="${meshes_file_direction}/link2.stl" scale="0.001 0.001 0.001"/>
         </geometry>
-        <material name="grey"/>
+        <material name="${visual_material}"/>
       </visual>
       <collision>
@@ -76,5 +76,5 @@
           <mesh filename="${meshes_file_direction}/link3.stl" scale="0.001 0.001 0.001"/>
         </geometry>
-        <material name="grey"/>
+        <material name="${visual_material}"/>
       </visual>
       <collision>
@@ -106,5 +106,5 @@
           <mesh filename="${meshes_file_direction}/link4.stl" scale="0.001 0.001 0.001"/>
         </geometry>
-        <material name="grey"/>
+        <material name="${visual_material}"/>
       </visual>
       <collision>
@@ -136,5 +136,5 @@
           <mesh filename="${meshes_file_direction}/link5.stl" scale="0.001 0.001 0.001"/>
         </geometry>
-        <material name="grey"/>
+        <material name="${visual_material}"/>
       </visual>
       <collision>
@@ -166,5 +166,5 @@
           <mesh filename="${meshes_file_direction}/gripper_left_palm.stl" scale="0.001 0.001 0.001"/>
         </geometry>
-        <material name="grey"/>
+        <material name="${visual_material}"/>
       </visual>
       <collision>
@@ -202,5 +202,5 @@
           <mesh filename="${meshes_file_direction}/gripper_right_palm.stl" scale="0.001 0.001 0.001"/>
         </geometry>
-        <material name="grey"/>
+        <material name="${visual_material}"/>
       </visual>
       <collision>
@@ -224,4 +224,5 @@
     </joint>
     <link name="${prefix}end_effector_link">
+      <xacro:if value="${show_tool_marker}">
       <visual>
         <origin xyz="0 0 0" rpy="0 0 0"/>
@@ -231,4 +232,5 @@
         <material name="red"/>
        </visual>
+      </xacro:if>
     </link>
   </xacro:macro>

File: turtlebot3_manipulation/turtlebot3_manipulation_description/xacro/orbbec_astra.urdf.xacro (robot description, xacro)
@@ -20,5 +20,6 @@
                        component_name:=''
                        use_tf_prefix:=True
-                       publish_internal_frames:=True">
+                       publish_internal_frames:=True
+                       leader_visuals:=False">
     <xacro:if value="${component_name == ''}">
       <xacro:property name="component_name" value="camera" />
@@ -43,4 +44,8 @@
     </joint>
     <link name="${component_name_underscore}astra_visual_frame">
+      <xacro:if value="${leader_visuals}">
+        <xacro:leader_depth_camera_visuals/>
+      </xacro:if>
+      <xacro:unless value="${leader_visuals}">
       <!-- Astra mesh is not present in this repository, so the model uses primitive visuals. -->
       <visual>
@@ -62,16 +67,24 @@
         </material>
       </visual>
+      </xacro:unless>
+      <!-- Move collision with the leader display housing, not the sensor TF. -->
+      <xacro:property name="camera_geometry_scale" value="${leader_camera_scale if leader_visuals else 1.0}"/>
+      <xacro:property name="camera_body_x" value="${leader_camera_body_x if leader_visuals else 0.0225-0.04/2.0}"/>
+      <xacro:property name="camera_body_z" value="${leader_camera_body_z if leader_visuals else 0.019+0.03/2.0}"/>
+      <xacro:property name="camera_pedestal_x" value="${leader_camera_pedestal_x if leader_visuals else 0.0235-0.06/2.0}"/>
+      <xacro:property name="camera_pedestal_bottom" value="${leader_camera_pedestal_bottom if leader_visuals else 0.0}"/>
+      <xacro:property name="camera_pedestal_height" value="${leader_camera_pedestal_height if leader_visuals else 0.019}"/>
       <!-- camera module collision -->
       <collision>
-        <origin xyz="${0.0225-0.04/2.0} 0.0 ${0.019+0.03/2.0}" rpy="0.0 0.0 0.0" />
+        <origin xyz="${camera_body_x} 0.0 ${camera_body_z}" rpy="0.0 0.0 0.0" />
         <geometry>
-          <box size="0.04 0.165 0.03" />
+          <box size="${0.04*camera_geometry_scale} ${0.165*camera_geometry_scale} ${0.03*camera_geometry_scale}" />
         </geometry>
       </collision>
       <!-- mounting base model collision -->
       <collision>
-        <origin xyz="${0.0235-0.06/2.0} 0.0 ${0.019/2.0}" rpy="0.0 0.0 0.0" />
+        <origin xyz="${camera_pedestal_x} 0.0 ${camera_pedestal_bottom+camera_pedestal_height/2.0}" rpy="0.0 0.0 0.0" />
         <geometry>
-          <box size="0.06 0.06 0.019" />
+          <box size="${0.06*camera_geometry_scale} ${0.06*camera_geometry_scale} ${camera_pedestal_height}" />
         </geometry>
       </collision>

File: turtlebot3_manipulation/turtlebot3_manipulation_description/xacro/turtlebot3_manipulation.urdf.xacro (robot description, xacro)
@@ -3,4 +3,6 @@
   <xacro:arg name="prefix" default="" />
   <xacro:arg name="use_sim" default="false" />
+  <xacro:arg name="leader_visuals" default="false" />
+  <xacro:property name="leader_visuals" value="$(arg leader_visuals)"/>
   <xacro:arg name="use_fake_hardware" default="false" />
   <xacro:arg name="fake_sensor_commands" default="false" />
@@ -11,4 +13,5 @@
   <xacro:arg name="eef_usb_camera_rpy" default="0.0 0.0 0.0" />
   <xacro:include filename="$(find turtlebot3_manipulation_description)/gazebo/materials.xacro" />
+  <xacro:include filename="leader_visuals.xacro"/>
   <xacro:include filename="$(find turtlebot3_manipulation_description)/xacro/turtlebot3_waffle_pi.urdf.xacro" />
   <xacro:include filename="$(find turtlebot3_manipulation_description)/gazebo/turtlebot3_waffle_pi.gazebo.xacro" />
@@ -18,22 +21,33 @@
   <xacro:turtlebot3_waffle_pi
     prefix="$(arg prefix)"
+    leader_visuals="${leader_visuals}"
     use_camera_driver_tf="$(arg use_camera_driver_tf)" />
+  <xacro:if value="${leader_visuals}">
+    <xacro:leader_tracks prefix="$(arg prefix)"/>
+    <xacro:leader_electronics prefix="$(arg prefix)"/>
+  </xacro:if>
+  <xacro:unless value="${leader_visuals}">
   <xacro:turtlebot3_waffle_pi_gazebo prefix="$(arg prefix)" />
+  </xacro:unless>
   <xacro:property name="support_radius" value="0.005" />
-  <xacro:property name="support_length" value="0.055" />
+  <xacro:property name="support_length" value="${leader_upper_support_length if leader_visuals else 0.055}" />
   <xacro:property name="support_center_z" value="0.145" />
   <xacro:macro name="plate_support" params="name x y">
+    <!-- Keep legacy support frames, move only display/collision geometry onto
+         the corrected three-piece stack. All robot/control TFs are unchanged. -->
+    <xacro:property name="support_visual_x" value="${(leader_tower_support_front_x if x > 0 else leader_support_back_x) - x if leader_visuals else 0}"/>
+    <xacro:property name="support_visual_z" value="${leader_upper_support_center_z - support_center_z if leader_visuals else 0}"/>
     <link name="$(arg prefix)${name}_link">
       <visual>
-        <origin xyz="0 0 0" rpy="0 0 0"/>
+        <origin xyz="${support_visual_x} 0 ${support_visual_z}" rpy="0 0 0"/>
         <geometry>
           <cylinder length="${support_length}" radius="${support_radius}"/>
         </geometry>
-        <material name="dark_grey">
-          <color rgba="0.2 0.2 0.2 1"/>
+        <material name="${'leader_support_metal' if leader_visuals else 'dark_grey'}">
+          <color rgba="${'0.65 0.67 0.69 1' if leader_visuals else '0.2 0.2 0.2 1'}"/>
         </material>
       </visual>
       <collision>
-        <origin xyz="0 0 0" rpy="0 0 0"/>
+        <origin xyz="${support_visual_x} 0 ${support_visual_z}" rpy="0 0 0"/>
         <geometry>
           <cylinder length="${support_length}" radius="${support_radius}"/>
@@ -57,4 +71,11 @@
   <xacro:plate_support name="support_back_right" x="-0.182" y="-0.05"/>
   <link name="$(arg prefix)upper_waffle_plate">
+    <xacro:if value="${leader_visuals}">
+      <!-- +28 mm visual offset aligns all layers at base x=-.064 while retaining
+           upper_waffle_plate_joint and the arm mounting transform. -->
+      <xacro:leader_mesh_visual file="upper_plate.stl" xyz="0.028 0 0"/>
+      <xacro:leader_box_visual size="0.030 0.026 0.004" xyz="0.105 0 0.007" color="leader_pcb"/>
+    </xacro:if>
+    <xacro:unless value="${leader_visuals}">
     <visual>
       <origin xyz="0 0 0" rpy="0 0 0"/>
@@ -66,8 +87,9 @@
       </material>
     </visual>
+    </xacro:unless>
     <collision>
-      <origin xyz="0 0 0" rpy="0 0 0"/>
+      <origin xyz="${'0.028 0 0' if leader_visuals else '0 0 0'}" rpy="0 0 0"/>
       <geometry>
-        <box size="0.290 0.136 0.01"/>
+        <box size="${leader_plate_size if leader_visuals else '0.290 0.136 0.01'}"/>
       </geometry>
     </collision>
@@ -81,13 +103,18 @@
     <parent link="$(arg prefix)base_link"/>
     <child link="$(arg prefix)upper_waffle_plate"/>
-    <origin xyz="-0.092 0.0 0.1775" rpy="0 0 0"/>
+    <origin xyz="-0.092 0.0 ${leader_upper_plate_z if leader_visuals else 0.1775}" rpy="0 0 0"/>
   </joint>
   <joint name="$(arg prefix)base_fixed" type="fixed">
     <parent link="$(arg prefix)base_link"/>
     <child link="$(arg prefix)link1"/>
-    <origin xyz="-0.092 0.0 0.178" rpy="0 0 0"/>
+    <!-- Latest user correction supersedes the standard XY display mount:
+         leader arm moves 36 mm rearward onto the added half plate. Keep
+         height .178 and RPY; hardware-default mount is not changed. -->
+    <origin xyz="${leader_arm_mount_x if leader_visuals else -0.092} 0.0 ${leader_arm_mount_z if leader_visuals else 0.178}" rpy="0 0 0"/>
   </joint>
-  <xacro:open_manipulator_x prefix="$(arg prefix)" />
+  <xacro:open_manipulator_x prefix="$(arg prefix)" visual_material="${'leader_arm' if leader_visuals else 'grey'}" show_tool_marker="${not leader_visuals}"/>
+  <xacro:unless value="${leader_visuals}">
   <xacro:open_manipulator_x_gazebo prefix="$(arg prefix)" />
+  </xacro:unless>
   <xacro:if value="$(arg use_eef_usb_camera)">
     <joint name="$(arg prefix)eef_usb_camera_joint" type="fixed">
@@ -97,4 +124,8 @@
     </joint>
     <link name="$(arg prefix)eef_usb_camera_link">
+      <xacro:if value="${leader_visuals}">
+        <xacro:leader_eef_camera_visuals/>
+      </xacro:if>
+      <xacro:unless value="${leader_visuals}">
       <visual>
         <origin xyz="0.025 0 0" rpy="0 0 0"/>
@@ -106,4 +137,5 @@
         </material>
       </visual>
+      </xacro:unless>
       <collision>
         <origin xyz="0.025 0 0" rpy="0 0 0"/>
@@ -137,4 +169,6 @@
     </xacro:if>
   </xacro:if>
+  <!-- A display-only profile must not expose a hardware/control plugin. -->
+  <xacro:unless value="${leader_visuals}">
   <xacro:turtlebot3_manipulation_system
     name="TurtleBot3ManipulationSystem" prefix="$(arg prefix)" use_sim="$(arg use_sim)"
@@ -147,3 +181,4 @@
     </plugin>
   </gazebo>
+  </xacro:unless>
 </robot>

File: turtlebot3_manipulation/turtlebot3_manipulation_description/xacro/turtlebot3_waffle_pi.urdf.xacro (robot description, xacro)
@@ -6,5 +6,5 @@
 -->
 <robot xmlns:xacro="http://www.ros.org/wiki/xacro">
-  <xacro:macro name="turtlebot3_waffle_pi" params="prefix use_camera_driver_tf:=false">
+  <xacro:macro name="turtlebot3_waffle_pi" params="prefix use_camera_driver_tf:=false leader_visuals:=false">
   <xacro:property
     name="meshes_file_direction"
@@ -17,4 +17,8 @@
   </joint>
   <link name="${prefix}base_link">
+    <xacro:if value="${leader_visuals}">
+      <xacro:leader_base_visuals/>
+    </xacro:if>
+    <xacro:unless value="${leader_visuals}">
     <visual>
       <origin xyz="-0.064 0 0.0" rpy="0 0 0"/>
@@ -24,8 +28,9 @@
       <material name="light_black"/>
     </visual>
+    </xacro:unless>
     <collision>
       <origin xyz="-0.064 0 0.047" rpy="0 0 0"/>
       <geometry>
-        <box size="0.266 0.266 0.094"/>
+        <box size="${'0.20155 0.13755 0.094' if leader_visuals else '0.266 0.266 0.094'}"/>
       </geometry>
     </collision>
@@ -45,4 +50,7 @@
   </joint>
   <link name="${prefix}wheel_left_link">
+    <!-- Wheel TFs/joint states are retained; tracked visuals are on base_link.
+         A whole belt cannot be rigidly rotated by wheel_left_joint. -->
+    <xacro:unless value="${leader_visuals}">
     <visual>
       <origin xyz="0 0 0" rpy="1.57 0 0"/>
@@ -58,4 +66,5 @@
       </geometry>
     </collision>
+    </xacro:unless>
     <inertial>
       <origin xyz="0 0 0" />
@@ -73,4 +82,5 @@
   </joint>
   <link name="${prefix}wheel_right_link">
+    <xacro:unless value="${leader_visuals}">
     <visual>
       <origin xyz="0 0 0" rpy="1.57 0 0"/>
@@ -86,4 +96,5 @@
       </geometry>
     </collision>
+    </xacro:unless>
     <inertial>
       <origin xyz="0 0 0" />
@@ -100,4 +111,5 @@
   </joint>
   <link name="${prefix}caster_back_right_link">
+    <xacro:unless value="${leader_visuals}">
     <collision>
       <origin xyz="0 0.001 0" rpy="0 0 0"/>
@@ -106,4 +118,5 @@
       </geometry>
     </collision>
+    </xacro:unless>
     <inertial>
       <origin xyz="0 0 0" />
@@ -120,4 +133,5 @@
   </joint>
   <link name="${prefix}caster_back_left_link">
+    <xacro:unless value="${leader_visuals}">
     <collision>
       <origin xyz="0 0.001 0" rpy="0 0 0"/>
@@ -126,4 +140,5 @@
       </geometry>
     </collision>
+    </xacro:unless>
     <inertial>
       <origin xyz="0 0 0" />
@@ -165,4 +180,8 @@
   </joint> -->
   <link name="${prefix}camera_plate_link">
+    <xacro:if value="${leader_visuals}">
+      <xacro:leader_mesh_visual file="camera_plate.stl"/>
+    </xacro:if>
+    <xacro:unless value="${leader_visuals}">
     <visual>
       <origin xyz="0 0 0" rpy="0 0 0"/>
@@ -172,8 +191,9 @@
       <material name="dark"/>
     </visual>
-    <collision>
-      <origin xyz="0 0 0" rpy="0 0 0"/>
-      <geometry>
-        <box size="0.266 0.266 0.005"/>
+    </xacro:unless>
+    <collision>
+      <origin xyz="0 0 0" rpy="0 0 0"/>
+      <geometry>
+        <box size="${leader_plate_size if leader_visuals else '0.266 0.266 0.005'}"/>
       </geometry>
     </collision>
@@ -187,5 +207,5 @@
     <parent link="${prefix}base_link"/>
     <child link="${prefix}camera_plate_link"/>
-    <origin xyz="-0.064 0.0 0.115" rpy="0 0 0"/>
+    <origin xyz="-0.064 0.0 ${leader_camera_plate_z if leader_visuals else 0.115}" rpy="0 0 0"/>
   </joint>
   <xacro:include filename="$(find turtlebot3_manipulation_description)/xacro/orbbec_astra.urdf.xacro" />
@@ -196,4 +216,5 @@
     robot_namespace="${prefix}"
     component_name="camera"
+    leader_visuals="${leader_visuals}"
     publish_internal_frames="${use_camera_driver_tf not in ['True', 'true', True]}" />
   </xacro:macro>
